File: brmecg.sch (EAGLE design)
At the start: 42 parts, among them U1 ADS1194CPAG

Commit message: Prepared for sex
Connections:
- net N$18 renamed DIN
- net N$19 renamed ~PWDN
- net N$20 renamed ~RESET
- net N$21 renamed START
- net N$23 renamed DAISY_IN
- net N$26 renamed DOUT
- net N$27 renamed ~DRDY
- removed net N$22: JP7.1, U1.SCLK
- removed net N$25: JP7.2, U1.~CS
- new net SCLK: JP7.2, U1.SCLK
- new net ~CS: JP7.1, U1.~CS
Other:
- moved on the sheet: JP7
