File: mindspy.sch (EAGLE design)
At the start: 39 parts, among them IC1 ADS1298, IC2 TPS7A4901, X1 DF9-31S, X2 STELLARIS-LAUNCHPADSTELLARIS-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

Commit message: almost final
Parts:
- added X10, X3, X5, X6, X7, X8, X9: MICRO-USB-AB-SCHIELD, molex:MICRO-USB-AB-SCHIELD
- X1: value DF9-31S -> MICRO-USB-AB-SCHIELD; device con-hirose:DF9-31S -> molex:MICRO-USB-AB-SCHIELD
Connections:
- net AIN1_N: now also X3CON.4; no longer X1.29
- net AIN1_P: now also X3CON.5; no longer X1.31
- net AIN2_N: now also X5CON.4; no longer X1.25
- net AIN2_P: now also X5CON.5; no longer X1.27
- net AIN3_N: now also X6CON.4; no longer X1.21
- net AIN3_P: now also X6CON.5; no longer X1.23
- net AIN4_N: now also X7CON.4; no longer X1.17
- net AIN4_P: now also X7CON.5; no longer X1.19
- net AIN5_N: now also X8CON.4; no longer X1.13
- net AIN5_P: now also X8CON.5; no longer X1.15
- net AIN6_N: now also X9CON.4; no longer X1.9
- net AIN6_P: now also X9CON.5; no longer X1.11
- net AIN7_N: now also X1CON.4; no longer X1.5
- net AIN7_P: now also X1CON.5; no longer X1.7
- net AIN8_N: now also X10CON.4; no longer X1.1
- net AIN8_P: now also X10CON.5; no longer X1.3
- net AVCM: now also X10CON.3, X1CON.3, X3CON.3, X5CON.3, X6CON.3, X7CON.3, X8CON.3, X9CON.3; no longer X1.18, X1.30
- net AVDD: now also X10CON.1, X1CON.1, X3CON.1, X5CON.1, X6CON.1, X7CON.1, X8CON.1, X9CON.1; no longer X1.20, X1.22, X1.24
- net AVSS: now also X10CON.2, X1CON.2, X3CON.2, X5CON.2, X6CON.2, X7CON.2, X8CON.2, X9CON.2; no longer X1.14, X1.16, X1.2, X1.4
- net RLDIN: no longer X1.8
- net RLDINV: no longer X1.10
- net RLDOUT: no longer X1.6
- net RLDREF: no longer X1.12
- net TEST_N: no longer X1.26
- net TEST_P: no longer X1.28
Other:
- moved on the sheet: SJ1, SJ2, SJ3, SJ4, SJ5

Commit message: errorneous previous commit
Parts:
- removed X10, X3, X5, X6, X7, X8, X9: MICRO-USB-AB-SCHIELD, molex:MICRO-USB-AB-SCHIELD
- added SJ6: (no value), jumper:SJ
- X1: value MICRO-USB-AB-SCHIELD -> DF9-31S; device molex:MICRO-USB-AB-SCHIELD -> con-hirose:DF9-31S
Connections:
- net AIN1_N: now also X1.29; no longer X3CON.4
- net AIN1_P: now also X1.31; no longer X3CON.5
- net AIN2_N: now also X1.25; no longer X5CON.4
- net AIN2_P: now also X1.27; no longer X5CON.5
- net AIN3_N: now also X1.21; no longer X6CON.4
- net AIN3_P: now also X1.23; no longer X6CON.5
- net AIN4_N: now also X1.17; no longer X7CON.4
- net AIN4_P: now also X1.19; no longer X7CON.5
- net AIN5_N: now also X1.13; no longer X8CON.4
- net AIN5_P: now also X1.15; no longer X8CON.5
- net AIN6_N: now also X1.9; no longer X9CON.4
- net AIN6_P: now also X1.11; no longer X9CON.5
- net AIN7_N: now also X1.5; no longer X1CON.4
- net AIN7_P: now also X1.7; no longer X1CON.5
- net AIN8_N: now also X1.1; no longer X10CON.4
- net AIN8_P: now also X1.3; no longer X10CON.5
- net AVCM: now also X1.22, X1.24, X1.26, X1.28, X1.30; no longer X10CON.3, X1CON.3, X3CON.3, X5CON.3, X6CON.3, X7CON.3, X8CON.3, X9CON.3
- net AVDD: now also X1.12, X1.14, X1.16, X1.18, X1.20; no longer X10CON.1, X1CON.1, X3CON.1, X5CON.1, X6CON.1, X7CON.1, X8CON.1, X9CON.1
- net AVSS: now also X1.10, X1.2, X1.4, X1.6, X1.8; no longer X10CON.2, X1CON.2, X3CON.2, X5CON.2, X6CON.2, X7CON.2, X8CON.2, X9CON.2
- net TEST_N: now also SJ6.1
- net TEST_P: now also SJ6.2
Other:
- moved on the sheet: SJ1, SJ2, SJ3, SJ4, SJ5

Commit message: .
Parts:
- removed L3: 10u, fabhack:L1210
Connections:
- net AVSS: no longer L3.2
- net DGND: no longer L3.1
Changed lines of the file:
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@@
 <part name="R2" library="rcl" deviceset="R-EU_" device="R0402"/>
 <part name="C2" library="rcl" deviceset="CPOL-EU" device="SMCA" value="10u"/>
-<part name="L3" library="fabhack" deviceset="L1210" device="" value="10u"/>
 <part name="X4" library="jumper" deviceset="JP3QE" device=""/>
 <part name="SUPPLY1" library="supply2" deviceset="VSS" device="" value="AVSS"/>
@@
 <instance part="C3" gate="G$1" x="170.18" y="132.08"/>
 <instance part="C4" gate="G$1" x="198.12" y="144.78"/>
-<instance part="SUPPLY7" gate="G$1" x="147.32" y="93.98"/>
+<instance part="SUPPLY7" gate="G$1" x="147.32" y="104.14"/>
 <instance part="SUPPLY10" gate="G$1" x="147.32" y="149.86"/>
 <instance part="SUPPLY8" gate="G$1" x="213.36" y="121.92"/>
@@
 <instance part="R2" gate="G$1" x="205.74" y="132.08" rot="MR90"/>
 <instance part="C2" gate="G$1" x="213.36" y="132.08"/>
-<instance part="L3" gate="G$1" x="154.94" y="101.6" rot="R90"/>
 <instance part="X4" gate="-1" x="190.5" y="109.22" rot="R270"/>
 <instance part="X4" gate="-2" x="177.8" y="109.22" rot="R270"/>
@@
 <pinref part="SUPPLY7" gate="G$1" pin="DGND"/>
 <pinref part="L2" gate="G$1" pin="1"/>
-<wire x1="147.32" y1="101.6" x2="147.32" y2="109.22" width="0.1524" layer="91"/>
+<wire x1="147.32" y1="106.68" x2="147.32" y2="109.22" width="0.1524" layer="91"/>
 <wire x1="147.32" y1="109.22" x2="147.32" y2="116.84" width="0.1524" layer="91"/>
 <wire x1="147.32" y1="116.84" x2="147.32" y2="124.46" width="0.1524" layer="91"/>
 <wire x1="142.24" y1="124.46" x2="147.32" y2="124.46" width="0.1524" layer="91"/>
 <junction x="147.32" y="124.46"/>
-<pinref part="L3" gate="G$1" pin="1"/>
-<junction x="147.32" y="101.6"/>
 <pinref part="X4" gate="-3" pin="1"/>
 <wire x1="142.24" y1="124.46" x2="142.24" y2="132.08" width="0.1524" layer="91"/>
@@
 <pinref part="L5" gate="G$1" pin="1"/>
 <junction x="147.32" y="109.22"/>
-<wire x1="147.32" y1="101.6" x2="147.32" y2="96.52" width="0.1524" layer="91"/>
 </segment>
 <segment>
@@
 <wire x1="205.74" y1="127" x2="205.74" y2="124.46" width="0.1524" layer="91"/>
 <junction x="205.74" y="124.46"/>
-<pinref part="L3" gate="G$1" pin="2"/>
-<wire x1="162.56" y1="101.6" x2="162.56" y2="109.22" width="0.1524" layer="91"/>
 <pinref part="L4" gate="G$1" pin="2"/>
 <wire x1="162.56" y1="109.22" x2="162.56" y2="116.84" width="0.1524" layer="91"/>
@@
 <junction x="162.56" y="116.84"/>
 <pinref part="L5" gate="G$1" pin="2"/>
-<junction x="162.56" y="109.22"/>
 <pinref part="IC2" gate="G$2" pin="GND@1"/>
 <wire x1="190.5" y1="134.62" x2="187.96" y2="134.62" width="0.1524" layer="91"/>

Commit message: use half-sized launchpad shield
Parts:
- X2: value STELLARIS-LAUNCHPADSTELLARIS-LAUNCHPAD -> STELLARIS-LAUNCHPAD-HALF; device fabhack:STELLARIS-LAUNCHPADSTELLARIS-LAUNCHPAD -> ti:STELLARIS-LAUNCHPAD-HALF
Changed lines of the file:
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@@
 <grid distance="0.1" unitdist="inch" unit="inch" style="lines" multiple="1" display="no" altdistance="0.01" altunitdist="inch" altunit="inch"/>
 <layers>
-<layer number="1" name="Top" color="4" fill="1" visible="no" active="no"/>
-<layer number="16" name="Bottom" color="1" fill="1" visible="no" active="no"/>
-<layer number="17" name="Pads" color="2" fill="1" visible="no" active="no"/>
-<layer number="18" name="Vias" color="2" fill="1" visible="no" active="no"/>
-<layer number="19" name="Unrouted" color="6" fill="1" visible="no" active="no"/>
-<layer number="20" name="Dimension" color="15" fill="1" visible="no" active="no"/>
-<layer number="21" name="tPlace" color="7" fill="1" visible="no" active="no"/>
-<layer number="22" name="bPlace" color="7" fill="1" visible="no" active="no"/>
-<layer number="23" name="tOrigins" color="15" fill="1" visible="no" active="no"/>
-<layer number="24" name="bOrigins" color="15" fill="1" visible="no" active="no"/>
-<layer number="25" name="tNames" color="7" fill="1" visible="no" active="no"/>
-<layer number="26" name="bNames" color="7" fill="1" visible="no" active="no"/>
-<layer number="27" name="tValues" color="7" fill="1" visible="no" active="no"/>
-<layer number="28" name="bValues" color="7" fill="1" visible="no" active="no"/>
+<layer number="1" name="Top" color="4" fill="1" visible="yes" active="no"/>
+<layer number="16" name="Bottom" color="1" fill="1" visible="yes" active="no"/>
+<layer number="17" name="Pads" color="2" fill="1" visible="yes" active="no"/>
+<layer number="18" name="Vias" color="2" fill="1" visible="yes" active="no"/>
+<layer number="19" name="Unrouted" color="6" fill="1" visible="yes" active="no"/>
+<layer number="20" name="Dimension" color="15" fill="1" visible="yes" active="no"/>
+<layer number="21" name="tPlace" color="7" fill="1" visible="yes" active="no"/>
+<layer number="22" name="bPlace" color="7" fill="1" visible="yes" active="no"/>
+<layer number="23" name="tOrigins" color="15" fill="1" visible="yes" active="no"/>
+<layer number="24" name="bOrigins" color="15" fill="1" visible="yes" active="no"/>
+<layer number="25" name="tNames" color="7" fill="1" visible="yes" active="no"/>
+<layer number="26" name="bNames" color="7" fill="1" visible="yes" active="no"/>
+<layer number="27" name="tValues" color="7" fill="1" visible="yes" active="no"/>
+<layer number="28" name="bValues" color="7" fill="1" visible="yes" active="no"/>
 <layer number="29" name="tStop" color="7" fill="3" visible="no" active="no"/>
 <layer number="30" name="bStop" color="7" fill="6" visible="no" active="no"/>
@@
 <layer number="35" name="tGlue" color="7" fill="4" visible="no" active="no"/>
 <layer number="36" name="bGlue" color="7" fill="5" visible="no" active="no"/>
-<layer number="37" name="tTest" color="7" fill="1" visible="no" active="no"/>
-<layer number="38" name="bTest" color="7" fill="1" visible="no" active="no"/>
+<layer number="37" name="tTest" color="7" fill="1" visible="yes" active="no"/>
+<layer number="38" name="bTest" color="7" fill="1" visible="yes" active="no"/>
 <layer number="39" name="tKeepout" color="4" fill="11" visible="no" active="no"/>
 <layer number="40" name="bKeepout" color="1" fill="11" visible="no" active="no"/>
@@
 <layer number="44" name="Drills" color="7" fill="1" visible="no" active="no"/>
 <layer number="45" name="Holes" color="7" fill="1" visible="no" active="no"/>
-<layer number="46" name="Milling" color="3" fill="1" visible="no" active="no"/>
-<layer number="47" name="Measures" color="7" fill="1" visible="no" active="no"/>
-<layer number="48" name="Document" color="7" fill="1" visible="no" active="no"/>
-<layer number="49" name="Reference" color="7" fill="1" visible="no" active="no"/>
-<layer number="50" name="dxf" color="7" fill="1" visible="no" active="no"/>
-<layer number="51" name="tDocu" color="7" fill="1" visible="no" active="no"/>
-<layer number="52" name="bDocu" color="7" fill="1" visible="no" active="no"/>
-<layer number="53" name="tGND_GNDA" color="7" fill="9" visible="no" active="no"/>
-<layer number="54" name="bGND_GNDA" color="1" fill="9" visible="no" active="no"/>
-<layer number="56" name="wert" color="7" fill="1" visible="no" active="no"/>
-<layer number="59" name="tCarbon" color="7" fill="1" visible="no" active="no"/>
-<layer number="60" name="bCarbon" color="7" fill="1" visible="no" active="no"/>
+<layer number="46" name="Milling" color="3" fill="1" visible="yes" active="no"/>
+<layer number="47" name="Measures" color="7" fill="1" visible="yes" active="no"/>
+<layer number="48" name="Document" color="7" fill="1" visible="yes" active="no"/>
+<layer number="49" name="Reference" color="7" fill="1" visible="yes" active="no"/>
+<layer number="50" name="dxf" color="7" fill="1" visible="yes" active="no"/>
+<layer number="51" name="tDocu" color="7" fill="1" visible="yes" active="no"/>
+<layer number="52" name="bDocu" color="7" fill="1" visible="yes" active="no"/>
+<layer number="53" name="tGND_GNDA" color="7" fill="9" visible="yes" active="no"/>
+<layer number="54" name="bGND_GNDA" color="1" fill="9" visible="yes" active="no"/>
+<layer number="56" name="wert" color="7" fill="1" visible="yes" active="no"/>
+<layer number="59" name="tCarbon" color="7" fill="1" visible="yes" active="no"/>
+<layer number="60" name="bCarbon" color="7" fill="1" visible="yes" active="no"/>
 <layer number="91" name="Nets" color="2" fill="1" visible="yes" active="yes"/>
 <layer number="92" name="Busses" color="1" fill="1" visible="yes" active="yes"/>
@@
 <parts>
 <part name="IC1" library="fabhack" deviceset="ADS1298" device=""/>
-<part name="X2" library="fabhack" deviceset="STELLARIS-LAUNCHPAD" device="STELLARIS-LAUNCHPAD"/>
+<part name="X2" library="ti" deviceset="STELLARIS-LAUNCHPAD-*" device="HALF"/>
 <part name="SUPPLY3" library="supply2" deviceset="DGND" device=""/>
 <part name="SUPPLY4" library="supply2" deviceset="DGND" device=""/>
