File: mindspy.sch (EAGLE design)
At the start: 40 parts, among them IC1 ADS1298IPAG, IC2 TPS7A4901, X1 DF9-31S, X2 STELLARIS-LAUNCHPAD-HALF

Commit message: Major changes
* placing improvements
 * labels on board
Parts:
- removed L4, L5: 10u, fabhack:L1210
Connections:
- net AVCM: now also X1.12, X1.18, X1.6; no longer X1.22, X1.26, X1.28
- net AVDD: now also X1.10, X1.22, X1.28, X1.4; no longer X1.12, X1.14, X1.18, X1.20
- net AVSS: now also X1.14, X1.20, X1.26; no longer L4.2, L5.2, X1.10, X1.4, X1.6
- net DGND: no longer L4.1, L5.1
Changed lines of the file:
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@@
 <part name="X4" library="jumper" deviceset="JP3QE" device=""/>
 <part name="SUPPLY1" library="supply2" deviceset="VSS" device="" value="AVSS"/>
-<part name="L4" library="fabhack" deviceset="L1210" device="" value="10u"/>
-<part name="L5" library="fabhack" deviceset="L1210" device="" value="10u"/>
 <part name="SJ6" library="jumper" deviceset="SJ" device=""/>
 <part name="SJ7" library="jumper" deviceset="SJ" device=""/>
@@
 <instance part="C3" gate="G$1" x="170.18" y="132.08"/>
 <instance part="C4" gate="G$1" x="198.12" y="144.78"/>
-<instance part="SUPPLY7" gate="G$1" x="147.32" y="104.14"/>
+<instance part="SUPPLY7" gate="G$1" x="147.32" y="121.92"/>
 <instance part="SUPPLY10" gate="G$1" x="147.32" y="149.86"/>
 <instance part="SUPPLY8" gate="G$1" x="215.9" y="121.92"/>
@@
 <instance part="X4" gate="-3" x="137.16" y="132.08" rot="R90"/>
 <instance part="SUPPLY1" gate="G$1" x="172.72" y="104.14"/>
-<instance part="L4" gate="G$1" x="154.94" y="116.84" rot="R90"/>
-<instance part="L5" gate="G$1" x="154.94" y="109.22" rot="R90"/>
 <instance part="SJ6" gate="1" x="20.32" y="106.68" rot="R180"/>
 <instance part="SJ7" gate="1" x="35.56" y="101.6" rot="R180"/>
@@
 <pinref part="SUPPLY7" gate="G$1" pin="DGND"/>
 <pinref part="L2" gate="G$1" pin="1"/>
-<wire x1="147.32" y1="106.68" x2="147.32" y2="109.22" width="0.1524" layer="91"/>
-<wire x1="147.32" y1="109.22" x2="147.32" y2="116.84" width="0.1524" layer="91"/>
-<wire x1="147.32" y1="116.84" x2="147.32" y2="124.46" width="0.1524" layer="91"/>
 <wire x1="142.24" y1="124.46" x2="147.32" y2="124.46" width="0.1524" layer="91"/>
 <junction x="147.32" y="124.46"/>
@@
 <wire x1="142.24" y1="132.08" x2="139.7" y2="132.08" width="0.1524" layer="91"/>
 <junction x="142.24" y="124.46"/>
-<pinref part="L4" gate="G$1" pin="1"/>
-<junction x="147.32" y="116.84"/>
-<pinref part="L5" gate="G$1" pin="1"/>
-<junction x="147.32" y="109.22"/>
 </segment>
 <segment>
@@
 <wire x1="208.28" y1="127" x2="208.28" y2="124.46" width="0.1524" layer="91"/>
 <junction x="208.28" y="124.46"/>
-<pinref part="L4" gate="G$1" pin="2"/>
-<wire x1="162.56" y1="109.22" x2="162.56" y2="116.84" width="0.1524" layer="91"/>
-<wire x1="162.56" y1="116.84" x2="162.56" y2="124.46" width="0.1524" layer="91"/>
-<junction x="162.56" y="116.84"/>
-<pinref part="L5" gate="G$1" pin="2"/>
 <pinref part="IC2" gate="G$2" pin="GND@1"/>
 <wire x1="190.5" y1="137.16" x2="187.96" y2="137.16" width="0.1524" layer="91"/>
@@
 </segment>
 <segment>
-<pinref part="X1" gate="DF9" pin="4"/>
-<wire x1="15.24" y1="55.88" x2="12.7" y2="53.34" width="0.1524" layer="91"/>
-<label x="12.7" y="53.34" size="1.27" layer="95" rot="R180" xref="yes"/>
-</segment>
-<segment>
-<pinref part="X1" gate="DF9" pin="6"/>
-<wire x1="15.24" y1="58.42" x2="12.7" y2="55.88" width="0.1524" layer="91"/>
-<label x="12.7" y="55.88" size="1.27" layer="95" rot="R180" xref="yes"/>
-</segment>
-<segment>
 <pinref part="X1" gate="DF9" pin="8"/>
 <wire x1="15.24" y1="60.96" x2="12.7" y2="58.42" width="0.1524" layer="91"/>
@@
 </segment>
 <segment>
-<pinref part="X1" gate="DF9" pin="10"/>
-<wire x1="15.24" y1="63.5" x2="12.7" y2="60.96" width="0.1524" layer="91"/>
-<label x="12.7" y="60.96" size="1.27" layer="95" rot="R180" xref="yes"/>
+<pinref part="X1" gate="DF9" pin="14"/>
+<wire x1="15.24" y1="68.58" x2="12.7" y2="66.04" width="0.1524" layer="91"/>
+<label x="12.7" y="66.04" size="1.27" layer="95" rot="R180" xref="yes"/>
+</segment>
+<segment>
+<pinref part="X1" gate="DF9" pin="20"/>
+<wire x1="15.24" y1="76.2" x2="12.7" y2="73.66" width="0.1524" layer="91"/>
+<label x="12.7" y="73.66" size="1.27" layer="95" rot="R180" xref="yes"/>
+</segment>
+<segment>
+<pinref part="X1" gate="DF9" pin="26"/>
+<wire x1="15.24" y1="83.82" x2="12.7" y2="81.28" width="0.1524" layer="91"/>
+<label x="12.7" y="81.28" size="1.27" layer="95" rot="R180" xref="yes"/>
 </segment>
 </net>
@@
 </segment>
 <segment>
-<pinref part="X1" gate="DF9" pin="20"/>
-<wire x1="15.24" y1="76.2" x2="12.7" y2="73.66" width="0.1524" layer="91"/>
-<label x="12.7" y="73.66" size="1.27" layer="95" rot="R180" xref="yes"/>
-</segment>
-<segment>
-<pinref part="X1" gate="DF9" pin="18"/>
-<wire x1="15.24" y1="73.66" x2="12.7" y2="71.12" width="0.1524" layer="91"/>
-<label x="12.7" y="71.12" size="1.27" layer="95" rot="R180" xref="yes"/>
-</segment>
-<segment>
 <pinref part="X1" gate="DF9" pin="16"/>
 <wire x1="15.24" y1="71.12" x2="12.7" y2="68.58" width="0.1524" layer="91"/>
@@
 </segment>
 <segment>
-<pinref part="X1" gate="DF9" pin="14"/>
-<wire x1="15.24" y1="68.58" x2="12.7" y2="66.04" width="0.1524" layer="91"/>
-<label x="12.7" y="66.04" size="1.27" layer="95" rot="R180" xref="yes"/>
-</segment>
-<segment>
-<pinref part="X1" gate="DF9" pin="12"/>
-<wire x1="15.24" y1="66.04" x2="12.7" y2="63.5" width="0.1524" layer="91"/>
-<label x="12.7" y="63.5" size="1.27" layer="95" rot="R180" xref="yes"/>
+<pinref part="X1" gate="DF9" pin="4"/>
+<wire x1="15.24" y1="55.88" x2="12.7" y2="53.34" width="0.1524" layer="91"/>
+<label x="12.7" y="53.34" size="1.27" layer="95" rot="R180" xref="yes"/>
+</segment>
+<segment>
+<pinref part="X1" gate="DF9" pin="10"/>
+<wire x1="15.24" y1="63.5" x2="12.7" y2="60.96" width="0.1524" layer="91"/>
+<label x="12.7" y="60.96" size="1.27" layer="95" rot="R180" xref="yes"/>
+</segment>
+<segment>
+<pinref part="X1" gate="DF9" pin="22"/>
+<wire x1="15.24" y1="78.74" x2="12.7" y2="76.2" width="0.1524" layer="91"/>
+<label x="12.7" y="76.2" size="1.27" layer="95" rot="R180" xref="yes"/>
+</segment>
+<segment>
+<pinref part="X1" gate="DF9" pin="28"/>
+<wire x1="15.24" y1="86.36" x2="12.7" y2="83.82" width="0.1524" layer="91"/>
+<label x="12.7" y="83.82" size="1.27" layer="95" rot="R180" xref="yes"/>
 </segment>
 </net>
@@
 </segment>
 <segment>
-<pinref part="X1" gate="DF9" pin="28"/>
-<wire x1="15.24" y1="86.36" x2="12.7" y2="83.82" width="0.1524" layer="91"/>
-<label x="12.7" y="83.82" size="1.27" layer="95" rot="R180" xref="yes"/>
-</segment>
-<segment>
-<pinref part="X1" gate="DF9" pin="26"/>
-<wire x1="15.24" y1="83.82" x2="12.7" y2="81.28" width="0.1524" layer="91"/>
-<label x="12.7" y="81.28" size="1.27" layer="95" rot="R180" xref="yes"/>
-</segment>
-<segment>
 <pinref part="X1" gate="DF9" pin="24"/>
 <wire x1="15.24" y1="81.28" x2="12.7" y2="78.74" width="0.1524" layer="91"/>
@@
 </segment>
 <segment>
-<pinref part="X1" gate="DF9" pin="22"/>
-<wire x1="15.24" y1="78.74" x2="12.7" y2="76.2" width="0.1524" layer="91"/>
-<label x="12.7" y="76.2" size="1.27" layer="95" rot="R180" xref="yes"/>
-</segment>
-</net>
+<pinref part="X1" gate="DF9" pin="6"/>
+<wire x1="15.24" y1="58.42" x2="12.7" y2="55.88" width="0.1524" layer="91"/>
+<label x="12.7" y="55.88" size="1.27" layer="95" rot="R180" xref="yes"/>
+</segment>
+<segment>
+<pinref part="X1" gate="DF9" pin="12"/>
+<wire x1="15.24" y1="66.04" x2="12.7" y2="63.5" width="0.1524" layer="91"/>
+<label x="12.7" y="63.5" size="1.27" layer="95" rot="R180" xref="yes"/>
+</segment>
+<segment>
+<pinref part="X1" gate="DF9" pin="18"/>
+<wire x1="15.24" y1="73.66" x2="12.7" y2="71.12" width="0.1524" layer="91"/>
+<label x="12.7" y="71.12" size="1.27" layer="95" rot="R180" xref="yes"/>
+</segment>
+</net>

Commit message: recent version of the prototype
Parts:
- added SJ8: (no value), jumper:SJ
Connections:
- new net AVDD2: C4.1, IC2G$1.OUT, R1.2, SJ8.1
- net AVDD: now also SJ8.2; no longer C4.1, IC2G$1.OUT, R1.2
Other:
- moved on the sheet: C2
Changed lines of the file:
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@@
 <part name="SJ6" library="jumper" deviceset="SJ" device=""/>
 <part name="SJ7" library="jumper" deviceset="SJ" device=""/>
+<part name="SJ8" library="jumper" deviceset="SJ" device=""/>
 </parts>
 <sheets>
@@
 <instance part="SUPPLY7" gate="G$1" x="147.32" y="121.92"/>
 <instance part="SUPPLY10" gate="G$1" x="147.32" y="149.86"/>
-<instance part="SUPPLY8" gate="G$1" x="215.9" y="121.92"/>
-<instance part="SUPPLY9" gate="G$1" x="215.9" y="149.86"/>
+<instance part="SUPPLY8" gate="G$1" x="218.44" y="121.92"/>
+<instance part="SUPPLY9" gate="G$1" x="218.44" y="149.86"/>
 <instance part="L1" gate="G$1" x="154.94" y="147.32" rot="R90"/>
 <instance part="L2" gate="G$1" x="154.94" y="124.46" rot="R90"/>
@@
 <instance part="R1" gate="G$1" x="208.28" y="142.24" rot="MR90"/>
 <instance part="R2" gate="G$1" x="208.28" y="132.08" rot="MR90"/>
-<instance part="C2" gate="G$1" x="215.9" y="132.08"/>
+<instance part="C2" gate="G$1" x="218.44" y="132.08"/>
 <instance part="X4" gate="-1" x="190.5" y="109.22" rot="R270"/>
 <instance part="X4" gate="-2" x="177.8" y="109.22" rot="R270"/>
@@
 <instance part="SJ6" gate="1" x="20.32" y="106.68" rot="R180"/>
 <instance part="SJ7" gate="1" x="35.56" y="101.6" rot="R180"/>
+<instance part="SJ8" gate="1" x="213.36" y="147.32"/>
 </instances>
 <busses>
@@
 <pinref part="SUPPLY8" gate="G$1" pin="VSS"/>
 <wire x1="190.5" y1="124.46" x2="208.28" y2="124.46" width="0.1524" layer="91"/>
-<junction x="215.9" y="124.46"/>
+<junction x="218.44" y="124.46"/>
 <pinref part="C2" gate="G$1" pin="-"/>
-<wire x1="208.28" y1="124.46" x2="215.9" y2="124.46" width="0.1524" layer="91"/>
-<wire x1="215.9" y1="124.46" x2="215.9" y2="127" width="0.1524" layer="91"/>
+<wire x1="208.28" y1="124.46" x2="218.44" y2="124.46" width="0.1524" layer="91"/>
+<wire x1="218.44" y1="124.46" x2="218.44" y2="127" width="0.1524" layer="91"/>
 <pinref part="R2" gate="G$1" pin="1"/>
 <wire x1="208.28" y1="127" x2="208.28" y2="124.46" width="0.1524" layer="91"/>
@@
 </segment>
 <segment>
-<pinref part="SUPPLY9" gate="G$1" pin="VCC"/>
-<pinref part="C2" gate="G$1" pin="+"/>
-<wire x1="215.9" y1="134.62" x2="215.9" y2="147.32" width="0.1524" layer="91"/>
-<pinref part="R1" gate="G$1" pin="2"/>
-<wire x1="208.28" y1="147.32" x2="215.9" y2="147.32" width="0.1524" layer="91"/>
-<junction x="215.9" y="147.32"/>
-<pinref part="IC2" gate="G$1" pin="OUT"/>
-<pinref part="C4" gate="G$1" pin="1"/>
-<wire x1="190.5" y1="147.32" x2="198.12" y2="147.32" width="0.1524" layer="91"/>
-<wire x1="198.12" y1="147.32" x2="208.28" y2="147.32" width="0.1524" layer="91"/>
-<junction x="198.12" y="147.32"/>
-<junction x="208.28" y="147.32"/>
-</segment>
-<segment>
 <pinref part="IC1" gate="G$1" pin="AVDD"/>
 <pinref part="IC1" gate="G$1" pin="AVDD@1"/>
@@
 <label x="12.7" y="83.82" size="1.27" layer="95" rot="R180" xref="yes"/>
 </segment>
+<segment>
+<pinref part="SUPPLY9" gate="G$1" pin="VCC"/>
+<pinref part="C2" gate="G$1" pin="+"/>
+<wire x1="218.44" y1="134.62" x2="218.44" y2="147.32" width="0.1524" layer="91"/>
+<pinref part="SJ8" gate="1" pin="2"/>
+<junction x="218.44" y="147.32"/>
+</segment>
 </net>
 <net name="AIN8_N" class="0">
@@
 </segment>
 </net>
+<net name="AVDD2" class="0">
+<segment>
+<pinref part="R1" gate="G$1" pin="2"/>
+<pinref part="IC2" gate="G$1" pin="OUT"/>
+<pinref part="C4" gate="G$1" pin="1"/>
+<wire x1="190.5" y1="147.32" x2="198.12" y2="147.32" width="0.1524" layer="91"/>
+<wire x1="198.12" y1="147.32" x2="208.28" y2="147.32" width="0.1524" layer="91"/>
+<junction x="198.12" y="147.32"/>
+<pinref part="SJ8" gate="1" pin="1"/>
+<junction x="208.28" y="147.32"/>
+</segment>
+</net>
