File: mindspy.brd (EAGLE design)
At the start: 45.7 x 50.8 mm, 38 parts, among them IC1 ADS1298IPAG, IC2 TPS7A4901, X1 DF9-31S, X2 STELLARIS-LAUNCHPAD-HALF

Commit message: recent version of the prototype
Parts:
- added SJ8: (no value), jumper:SJ
- moved C3 2.02 mm to (4.17, 16.0)
- moved C4 2.02 mm to (13.9, 15.4)
- moved C5 2.02 mm to (3.22, 14.5)
- moved IC2 2.02 mm to (8.62, 15.7)
- moved R1 2.02 mm to (12.6, 15.1)
- moved R2 2.02 mm to (12.6, 17.3)
Connections:
- new net AVDD2: C4.1, IC2.1, R1.2, SJ8.1
- net AVDD: now also SJ8.2; no longer C4.1, IC2.1, R1.2
Routing:
- net AVDD2: track 0.00 -> 5.00 mm
- net AVDD: track 30.7 -> 26.8 mm
- net N$22: track 7.51 -> 8.06 mm
