File: hw/brmeeg.brd (EAGLE design)
At the start: 52.1 x 24.3 mm, 42 parts, among them U1 ADS1194CPAG

Commit message: final updates to ADC board
Parts:
- moved JP13 8.27 mm to (2.44, 21.4)
- moved C2 0.90 mm to (40.6, 20.8)
- moved C9 0.90 mm to (40.8, 22.3)
- moved C15 0.56 mm to (4.24, 10.2)
- moved C16 0.56 mm to (4.24, 6.74)
- moved C11 0.56 mm to (38.2, 2.87)
- moved C12 0.56 mm to (40.1, 2.87)
- moved C13 0.56 mm to (27.6, 2.71)
- moved C14 0.56 mm to (31.2, 18.4)
- moved C18 0.56 mm to (6.99, 6.75)
- moved C20 0.56 mm to (8.39, 6.75)
- moved C21 0.56 mm to (7.88, 15.1)
- moved C22 0.56 mm to (10.6, 5.18)
- moved C23 0.56 mm to (12.7, 21.4)
- moved C24 0.56 mm to (19.5, 22.9)
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Routing:
- net GND: track 56.8 -> 65.6 mm
- net +3V3/1: track 4.56 -> 13.1 mm
- net SCLK: track 7.78 -> 6.64 mm
- net DAISY_IN: track 9.82 -> 8.80 mm
- net ~RESET: track 7.48 -> 6.51 mm
- net START: track 5.96 -> 5.00 mm
- net ~PWDN: track 9.54 -> 8.68 mm
- net ~CS: track 5.75 -> 4.95 mm
- net DIN: track 11.6 -> 10.8 mm
- net ~DRDY: track 11.9 -> 11.2 mm
- net DOUT: track 11.4 -> 10.7 mm
- net N$8: track 5.04 -> 4.51 mm
Other:
- board size 52.1 x 24.3 mm -> 49.6 x 25.6 mm
- board text added: "MindSpy.org"
- board text added: "ver 0.1"

Commit message: final updates to ADC board
Routing:
- net +3V3: track 43.9 -> 41.2 mm, vias 2 -> 0
Changed lines of the file:
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@@
 <layers>
 <layer number="1" name="Top" color="4" fill="1" visible="yes" active="yes"/>
-<layer number="16" name="Bottom" color="1" fill="1" visible="no" active="yes"/>
+<layer number="16" name="Bottom" color="1" fill="1" visible="yes" active="yes"/>
 <layer number="17" name="Pads" color="2" fill="1" visible="yes" active="yes"/>
 <layer number="18" name="Vias" color="2" fill="1" visible="yes" active="yes"/>
-<layer number="19" name="Unrouted" color="6" fill="1" visible="yes" active="yes"/>
+<layer number="19" name="Unrouted" color="6" fill="1" visible="no" active="yes"/>
 <layer number="20" name="Dimension" color="15" fill="1" visible="yes" active="yes"/>
 <layer number="21" name="tPlace" color="7" fill="1" visible="no" active="yes"/>
@@
 <wire x1="42.75" y1="16.2592" x2="42.75" y2="16.5" width="0.254" layer="1"/>
 <wire x1="42.75" y1="16.5" x2="42.75" y2="19.75" width="0.4064" layer="1"/>
-<via x="42.75" y="19.75" extent="1-16" drill="0.6"/>
-<wire x1="42.75" y1="19.75" x2="40.0012" y2="19.75" width="0.4064" layer="16"/>
-<via x="40.0012" y="19.75" extent="1-16" drill="0.6"/>
+<wire x1="42.75" y1="19.75" x2="42.75" y2="19.75" width="0" layer="19" extent="1-16"/>
+<wire x1="42.75" y1="19.75" x2="40.0012" y2="19.75" width="0" layer="19" extent="1-16"/>
+<wire x1="40.0012" y1="19.75" x2="40.0012" y2="19.75" width="0" layer="19" extent="1-16"/>
 <wire x1="22.58" y1="18.28" x2="22.58" y2="18.33" width="0.4064" layer="1"/>
 <wire x1="22.58" y1="18.33" x2="24.5" y2="20.25" width="0.6096" layer="1"/>
