File: hw/stellaris/mindspy.brd (EAGLE design)
At the start: 69.5 x 53.3 mm, 43 parts, among them IC1 ADS1298, IC3 MCP1703CB, X1 DF9-31S, X2 STELLARIS-LAUNCHPADSTELLARIS-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

Commit message: Major modifications.
Parts:
- removed C15, C19: 1u, rcl:C0805K
- removed C16, C20: 0.1u, rcl:C0603K
- removed IC3: MCP1703CB, linear:SOT23
- removed SJ10, SJ6, SJ7, SJ8, SJ9: (no value), jumper:SJ
- removed X3: (no value), jumper:JP8Q
- added IC2: TPS7A4901, fabhack:MSOP08
- added L3: 10u, fabhack:L1210K
- added R1, R2: (no value), rcl:R0402
- added X4: (no value), jumper:JP3Q
- C1, C2, C5: device rcl:SMC_B -> rcl:SMC_A
- C10, C11, C12, C14, C18, C22, C8, C9: device rcl:C0603K -> rcl:C0402
- C13, C17, C21, C23: device rcl:C0805K -> rcl:C0402
- C3, C4: device rcl:C0603K -> rcl:C0603
- C6: device rcl:C0805K -> rcl:C0805
- C7: device rcl:C1206K -> rcl:C0805
- L1, L2: device rcl:L1812 -> fabhack:L1210K
- SJ1, SJ2: device jumper:SJ_2 -> jumper:SJ
- moved C10 42.0 mm to (44.1, 24.1), turned to 270 degrees
- moved C23 41.7 mm to (41.0, 40.0)
- moved C14 36.5 mm to (44.8, 38.7), turned to 180 degrees
- moved C22 35.5 mm to (39.1, 24.8), turned to 180 degrees
- moved C13 34.7 mm to (44.8, 40.0), turned to 180 degrees
- moved C18 33.7 mm to (39.1, 39.4), turned to 90 degrees
- moved C21 33.2 mm to (39.1, 23.5), turned to 180 degrees
- moved C17 31.8 mm to (38.1, 39.4), turned to 90 degrees
- moved C12 30.3 mm to (41.0, 38.7)
- moved C7 27.3 mm to (45.7, 24.8), turned to 270 degrees
- moved C6 26.6 mm to (42.2, 22.5), turned to 270 degrees
- moved C11 26.1 mm to (36.8, 39.4), turned to 270 degrees
- moved C9 25.8 mm to (42.2, 24.8)
- moved C4 25.4 mm to (40.0, 16.8), turned to 90 degrees
- moved C5 25.2 mm to (26.4, 16.5)
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Connections:
- net AIN1N renamed AIN1_N
- net AIN1P renamed AIN1_P
- net AIN2N renamed AIN2_N
- net AIN2P renamed AIN2_P
- net AIN3N renamed AIN3_N
- net AIN3P renamed AIN3_P
- net AIN4N renamed AIN4_N
- net AIN4P renamed AIN4_P
- net AIN5N renamed AIN5_N
- net AIN5P renamed AIN5_P
- net AIN6N renamed AIN6_N
- net AIN6P renamed AIN6_P
- net AIN7N renamed AIN7_N
- net AIN7P renamed AIN7_P
- net AIN8N renamed AIN8_N
- net AIN8P renamed AIN8_P
- removed net AGND: C15.2, C16.2, C17.2, C18.2, C19.2, C20.2, C21.1, C22.1, X1.4, X3.11
- removed net DAISY: IC1.41, SJ2.2
- removed net DOUT: IC1.43, SJ1.2
- removed net N$10: SJ7.1, X3.4
- removed net N$11: SJ6.1, X3.5
- removed net N$12: SJ5.1, X3.6
- removed net N$13: SJ8.1, X3.3
- removed net N$14: SJ3.1, X3.8
- removed net N$15: SJ10.1, X3.1
- removed net N$16: SJ10.2, SJ2.3, SJ4.2, SJ6.2, SJ8.2
- removed net N$18: SJ1.1, SJ3.2, SJ5.2, SJ7.2, SJ9.2
- removed net N$9: SJ4.1, X3.7
- new net !CS1: SJ1.2, X2.PD1
- new net !CS2: SJ2.2
- new net !CS3: SJ3.2
- new net !CS4: SJ4.2
- new net !CS5: SJ5.2
- new net AVCM: X1.18, X1.30, X4.2
- new net N$19: C4.2, IC2.2, R1.1, R2.2
- new net N$22: C5.+, IC2.5, IC2.8, L1.2
- new net PWREN: X2.PB0
- net !CS: now also SJ1.1, SJ2.1, SJ3.1, SJ4.1, SJ5.1; no longer X2.PD1
- net AVDD: now also C2.+, C4.1, IC2.1, R1.2, X1.20, X1.22, X1.24, X4.1; no longer C5.+, L1.2, X1.30, X3.13
- net AVSS: now also C17.2, C18.2, C2.-, C21.1, C22.1, C3.2, IC2.4, L3.2, R2.1, X1.14, X1.16, X1.4, X4.3, X4.4; no longer C15.1, C16.1, C19.1, C20.1, X3.14
- net CLK: now also X2.PB3; no longer X3.10
- net DGND: now also IC1.41, L3.1, X4.5; no longer C2.-, C3.1, C4.2, IC3.1, SJ2.1, X1.22, X3.15
- net DVDD: now also L1.1, X4.6; no longer C3.2, IC3.3, X1.24, X3.16
- net GPIO1: no longer X1.14
- net GPIO2: no longer X1.16
- net GPIO3: no longer X1.18
- net GPIO4: no longer X1.20
- net MISO: now also IC1.43; no longer SJ1.3
- net N$3: now also C3.1, IC2.6; no longer C2.+, C4.1, IC3.2, L1.1
- net N$8: now also IC2.P$1, IC2.P$2, IC2.P$3, IC2.P$4, IC2.P$5; no longer SJ9.1, X3.2
Routing:
- net DVDD: track 0.00 -> 74.5 mm, vias 0 -> 2
- net AVDD: track 0.00 -> 32.0 mm
- net DGND: track 0.00 -> 18.7 mm
- net !CS: track 0.00 -> 15.3 mm
- net AVCM: track 0.00 -> 14.2 mm
- net N$22: track 0.00 -> 10.4 mm
- net AIN8_N: track 0.00 -> 7.57 mm
- net AIN1_P: track 0.00 -> 7.57 mm
- net AIN8_P: track 0.00 -> 7.35 mm
- net AIN1_N: track 0.00 -> 7.35 mm
- net AIN7_N: track 0.00 -> 7.14 mm
- net AIN2_P: track 0.00 -> 7.14 mm
- net AIN7_P: track 0.00 -> 6.91 mm
- net AIN2_N: track 0.00 -> 6.91 mm
- net AIN6_N: track 0.00 -> 6.74 mm
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- added copper zone on layer 1, net AVSS
- added copper zone on layer 16, net AVSS
- added copper zone on layer 1, net DGND
- added copper zone on layer 16, net DGND

Commit message: digital prat completed
Parts:
- added L4, L5: 10u, fabhack:L1210K
- moved SJ5 5.68 mm to (54.6, 29.2), flipped to the bottom, turned to 270 degrees
- moved SJ1 5.55 mm to (55.9, 33.0), turned to 90 degrees
- moved L3 5.25 mm to (27.2, 45.8), turned to 225 degrees
- moved SJ3 4.07 mm to (58.4, 29.2), flipped to the bottom, turned to 270 degrees
- moved SJ4 2.71 mm to (56.5, 29.2), flipped to the bottom, turned to 270 degrees
- moved C21 2.56 mm to (36.8, 24.8), turned to 0 degrees
- moved C4 2.56 mm to (37.5, 17.1)
- moved R1 2.54 mm to (36.2, 16.8)
- moved C11 2.29 mm to (35.6, 37.5), turned to 0 degrees
- moved IC2 2.22 mm to (32.4, 17.5)
- moved X4 2.22 mm to (41.9, 14.0)
- moved C6 2.22 mm to (42.2, 20.3), turned to 315 degrees
- moved C18 2.01 mm to (37.1, 38.7), turned to 180 degrees
- moved C3 1.93 mm to (27.9, 17.8)
- moved C8 1.59 mm to (40.1, 22.3), turned to 225 degrees
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Connections:
- removed net N$8: IC2.P$1, IC2.P$2, IC2.P$3, IC2.P$4, IC2.P$5
- removed net PWREN: X2.PB0
- net !CS1: now also X2.PA3; no longer X2.PD1
- net !CS2: now also X2.PF4
- net !CS3: now also X2.PE1
- net !CS4: now also X2.PB4
- net !CS5: now also X2.PD3
- net !DRDY: now also X2.PC6; no longer X2.PE1
- net !RESET: now also X2.PA6; no longer X2.PE3
- net AVSS: now also IC2.NC@0, IC2.NC@1, IC2.NC@2, IC2.NC@3, IC2.NC@4, IC2.PWR@1, IC2.PWR@2, L4.2, L5.2
- net CLK: now also X2.PE3; no longer X2.PB3
- net DGND: now also L4.1, L5.1
- net GPIO1: now also X2.PD7; no longer X2.PB4
- net GPIO2: now also X2.PB6; no longer X2.PA5
- net GPIO3: now also X2.PC7; no longer X2.PA6
- net GPIO4: now also X2.PB7; no longer X2.PA7
- net MISO: now also X2.PA4; no longer X2.PD2
- net MOSI: now also X2.PA5; no longer X2.PD3
- net SCLK: now also X2.PA2; no longer X2.PD0
- net START: now also X2.PA7; no longer X2.PE4
Routing:
- net !CS4: track 0.00 -> 34.8 mm
- net START: track 0.00 -> 34.2 mm
- net AVDD: track 32.0 -> 65.8 mm, vias 0 -> 4
- net !CS5: track 0.00 -> 32.3 mm
- net !CS3: track 0.00 -> 32.0 mm
- net !RESET: track 1.63 -> 32.8 mm
- net MOSI: track 1.36 -> 31.8 mm
- net CLK: track 0.00 -> 30.3 mm
- net !PWDN: track 1.49 -> 29.3 mm
- net SCLK: track 1.22 -> 25.3 mm
- net !CS1: track 0.00 -> 23.7 mm
- net GPIO2: track 1.44 -> 22.8 mm
- net MISO: track 1.30 -> 22.4 mm
- net GPIO4: track 1.39 -> 21.8 mm
- net GPIO1: track 1.17 -> 20.2 mm
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
Commit message: minor change
Parts:
- moved SJ1 2.54 mm to (53.3, 33.0)
- moved SJ2 2.54 mm to (51.4, 33.0)
- moved C21 1.31 mm to (36.5, 23.5)
- moved SJ3 0.95 mm to (57.5, 29.2)
- moved SJ4 0.95 mm to (55.6, 29.2)
- moved SJ5 0.95 mm to (53.7, 29.2)
Connections:
- net TESTN renamed TEST_N
- net TESTP renamed TEST_P
Routing:
- net TEST_N: track 0.00 -> 4.92 mm
- net TEST_P: track 0.00 -> 4.52 mm
- net !CS2: track 14.0 -> 17.4 mm
- net !CS1: track 23.7 -> 26.9 mm
- net GPIO2: track 22.8 -> 20.2 mm
- net AVDD: track 65.8 -> 63.2 mm, vias 4 -> 3
- net GPIO3: track 19.2 -> 17.1 mm
- net GPIO4: track 21.8 -> 20.3 mm
- net !CS: track 18.5 -> 17.0 mm
- net !DRDY: track 18.2 -> 17.0 mm
- net !RESET: track 32.8 -> 31.6 mm
- net !CS3: track 32.0 -> 30.9 mm
- net MISO: track 22.4 -> 21.3 mm
- net CLK: track 30.3 -> 29.2 mm
- net !CS4: track 34.8 -> 34.1 mm
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Other:
- board size 69.5 x 53.3 mm -> 68.6 x 53.3 mm
